File: hardware/pt_board/pt_board.kicad_sch (KiCad schematic)
At the start: 7 parts, among them J2 IR Blaster 3.5mm, J3 LANC 2.5mm, U1 ESP32-S3-WROOM-1, U2 AZ1117-3.3

Commit message: added rgb led to schematic
Parts:
- added D1: LED_RGBA, symbol Device:LED_RGBA
- U2: value AZ1117-3.3 -> AZ1117I-3.3
Changed lines of the file:
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@@
       (effects (font (size 1.27 1.27)))
     )
-    (property "Value" "AZ1117-3.3" (at 78.74 13.97 0)
+    (property "Value" "AZ1117I-3.3" (at 78.74 13.97 0)
       (effects (font (size 1.27 1.27)))
     )
@@
         )
       )
+    )
+  )
+  (symbol (lib_id "Device:LED_RGBA") (at 69.85 76.2 0) (unit 1)
+    (in_bom yes) (on_board yes) (dnp no) (fields_autoplaced)
+    (property "Reference" "D1" (at 69.85 63.5 0)
+      (effects (font (size 1.27 1.27)))
+    )
+    (property "Value" "LED_RGBA" (at 69.85 66.04 0)
+      (effects (font (size 1.27 1.27)))
+    )
+    (property "Footprint" "" (at 69.85 77.47 0)
+      (effects (font (size 1.27 1.27)) hide)
+    )
+    (property "Datasheet" "~" (at 69.85 77.47 0)
+      (effects (font (size 1.27 1.27)) hide)
+    )
+    (pin "1")
+    (pin "2")
+    (pin "3")
+    (pin "4")
+    (instances
+      (project "pt_board"
+        (path "/98360be2-1f1b-4904-9f9a-1928b68df9c7"
+          (reference "D1") (unit 1)
+        )
+      )
